File: QPOL.kicad_pcb (KiCad board)
At the start: 2 copper layers, 142.6 x 128.4 mm, 105 parts, among them J1 Conn_01x10_Pin, J10 AudioJack2, J11 AudioJack2, J15 Conn_02x05_Odd_Even, J2 Conn_01x03_Pin, J3 Conn_01x03_Pin, J4 AudioJack2, J5 Conn_01x10_Pin, J6 AudioJack2, J9 AudioJack2, Q2 BC857, SW1 SW_SPDT, U1 TL074, U2 TL074, U3 LM13700, U4 LM13700, U5 TL074, U6 TL072

Commit message: Add files via upload
Parts:
- removed the ? at (162.5, 130.9)
- removed the ? at (98.9, 129.7)
- added ?: , , F.Cu at (159.8, 132.5)
- added ?: , , F.Cu at (104.1, 134.6)
- added J7: Conn_01x03_Pin, Connector_PinSocket_2.54mm:PinSocket_1x03_P2.54mm_Vertical, B.Cu at (140.4, 104.4)
- C10, C2, C3, C9: value 10n -> 1n
- J5: moved to F.Cu
- R26: value 10k -> 4k7
- moved J5 60.9 mm to (140.6, 108.3), turned to 0 degrees
- moved J1 58.5 mm to (85.0, 110.4)
- moved J11 7.12 mm to (111.0, 141.2)
- moved D5 7.12 mm to (90.7, 70.6)
- moved J10 7.12 mm to (111.1, 87.2)
- moved J2 7.12 mm to (84.7, 79.9)
- moved J6 7.12 mm to (111.0, 69.4)
- moved J9 7.12 mm to (90.8, 104.1)
- moved R25 7.12 mm to (111.2, 123.2)
- moved R26 7.12 mm to (94.6, 70.8)
- moved RV4 7.12 mm to (88.3, 94.7)
- moved RV6 7.12 mm to (98.4, 129.6)
- moved RV5 7.12 mm to (88.2, 62.0)
- moved RV7 7.12 mm to (108.5, 62.0)
- moved D6 7.12 mm to (109.8, 129.9)
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Connections:
- R61 pad 2: INQAP -> Net-(J7-Pin_2)
Routing:
- net INQAP: track 73.9 -> 91.0 mm, vias 5 -> 6
- net Net-(J7-Pin_2): track 0.00 -> 11.0 mm
- net GND: track 37.4 -> 46.5 mm, vias 9 -> 11
- net IN: track 57.3 -> 62.4 mm, vias 1 -> 2
- net Net-(U5C-+): track 21.7 -> 22.7 mm
- net FDBKIN: track 70.8 -> 70.1 mm
- net FDBKATTEN: track 45.9 -> 45.3 mm, vias 1 -> 3
Other:
- board size 142.6 x 128.4 mm -> 139.9 x 128.4 mm
- board text added: "Mixed Direct"
