File: QPOL.kicad_sch (KiCad schematic)
At the start: 55 parts, among them J1 Conn_01x10_Pin, J10 AudioJack2, J11 AudioJack2, J15 Conn_02x05_Odd_Even, J2 Conn_01x03_Pin, J3 Conn_01x03_Pin, J4 AudioJack2, J5 Conn_01x10_Pin, J6 AudioJack2, J9 AudioJack2, Q2 BC857, SW1 SW_SPDT, U1 TL074, U2 TL074, U3 LM13700, U4 LM13700, U5 TL074, U6 TL072

Commit message: Add files via upload
Parts:
- added J7: Conn_01x03_Pin, Connector_PinSocket_2.54mm:PinSocket_1x03_P2.54mm_Vertical, symbol Connector:Conn_01x03_Pin
Connections:
- net IN: now also J7.1 (Pin_1)
- net INQAP: now also J7.3 (Pin_3); no longer R61.2
- new net: J7.2 (Pin_2), R61.2
- no-connect marks 0 -> 2
Other:
- moved on the sheet: J1, J2
